Commit message: right arm IK working

File: data/ravenII_2arm.urdf (robot description, URDF)
Before this commit: robot raven_2, 19 links, 18 joints
Links:
- added link tool_R
Joints:
- added joint grasper_yaw_R: type revolute, parent wrist_R, child tool_R, origin xyz=0.012 0 0 rpy=-1.5707963267948966 0 0, axis 0 0 1, limit lower=-2 upper=2 effort=1000.0 velocity=.5
