Commit message: added raven vision, updated urdfs
--HG--
rename : raven_2_params/data/ravenII_2arm.urdf => raven_2_params/data/ravenII_both_arm.urdf

File: raven_2_params/data/ravenII_gold_arm.urdf (robot description, URDF)
Before this commit: robot raven_2, 20 links, 19 joints
Links:
- removed link base_link_R
- removed link grasper1_R
- removed link grasper2_R
- removed link instrument_shaft_R
- removed link link1_R
- removed link link2_R
- removed link link3_R
- removed link tool_R
- removed link wrist_R
- added link grasper1_tip_L
- added link grasper2_tip_L
- added link tool_base_L
- added link tool_tip_L
Joints:
- removed joint camera_L
- removed joint camera_R
- removed joint elbow_R
- removed joint grasper_joint_1_R
- removed joint grasper_joint_2_R
- removed joint grasper_yaw_R
- removed joint insertion_R
- removed joint shoulder_R
- removed joint tool_roll_R
- removed joint wrist_joint_R
- added joint base_mount_L: type fixed, parent 0_link, child base_link_L, origin xyz=0.0 0.00 0 rpy=0 0 -1.5707963267948966, limit lower=0.0 upper=3.1415 effort=1000.0 velocity=0.5
- added joint grasper1_tip_L: type fixed, parent grasper1_L, child grasper1_tip_L, origin xyz=0.02 0 0 rpy=0 0 0, limit lower=0.0 upper=3.1415 effort=1000.0 velocity=0.5
- added joint grasper2_tip_L: type fixed, parent grasper2_L, child grasper2_tip_L, origin xyz=0.02 0 0 rpy=0 0 0, limit lower=0.0 upper=3.1415 effort=1000.0 velocity=0.5
- added joint tool_base_to_main_L: type fixed, parent tool_base_L, child tool_L, origin xyz=0.01 0 0 rpy=0 0 0, limit lower=0.0 upper=3.1415 effort=1000.0 velocity=0.5
- added joint tool_base_to_tip_L: type fixed, parent tool_base_L, child tool_tip_L, origin xyz=0.02 0 0 rpy=0 0 0, limit lower=0.0 upper=3.1415 effort=1000.0 velocity=0.5
- joint grasper_yaw_L: child tool_L -> tool_base_L
- joint world_to_0_link: origin xyz=0.0 0.00 0 rpy=0 0 1.5707963267948966 -> xyz=.211 -.25071 .235 rpy=0 0 1.5707963267948966
