Commit message: fixed green arm base position, added frame to urdf

File: raven_2_params/data/ravenII_green_arm.urdf (robot description, URDF)
Before this commit: robot raven_2, 16 links, 15 joints
Links:
- added link frame_base_support_L; visual box size=0.4 0.05 0.025
- added link frame_base_support_R; visual box size=0.4 0.05 0.025
- added link frame_bottom_B; visual box size=0.70 0.025 0.025
- added link frame_bottom_F; visual box size=0.7 0.025 0.025
- added link frame_bottom_L; visual box size=0.40 0.025 0.025
- added link frame_bottom_R; visual box size=0.40 0.025 0.025
- added link frame_top_B; visual box size=0.70 0.025 0.025
- added link frame_top_F; visual box size=0.7 0.025 0.025
- added link frame_top_L; visual box size=0.40 0.025 0.025
- added link frame_top_R; visual box size=0.40 0.025 0.025
- added link frame_vertical_LB; visual box size=0.10 0.025 0.025
- added link frame_vertical_LF; visual box size=0.10 0.025 0.025
- added link frame_vertical_RB; visual box size=0.10 0.025 0.025
- added link frame_vertical_RF; visual box size=0.10 0.025 0.025
- link base_link_R: geometry visual mesh filename=package://raven_2_params/data/right_arm/base_w_motors.dae
Joints:
- added joint world_to_frame_base_support_L: type fixed, parent world, child frame_base_support_L, origin xyz=0.1315 0.05 0.2 rpy=0 -1.5707963267948966 0
- added joint world_to_frame_base_support_R: type fixed, parent world, child frame_base_support_R, origin xyz=0.1315 -0.7 0.2 rpy=0 -1.5707963267948966 0
- added joint world_to_frame_bottom_B: type fixed, parent world, child frame_bottom_B, origin xyz=0.4125 -0.325 0.0125 rpy=0 0 -1.5707963267948966
- added joint world_to_frame_bottom_F: type fixed, parent world, child frame_bottom_F, origin xyz=-0.0125 -0.325 0.0125 rpy=0 0 -1.5707963267948966
- added joint world_to_frame_bottom_L: type fixed, parent world, child frame_bottom_L, origin xyz=0.20 0.0125 0.0125 rpy=0 0 0
- added joint world_to_frame_bottom_R: type fixed, parent world, child frame_bottom_R, origin xyz=0.20 -0.6625 0.0125 rpy=0 0 0
- added joint world_to_frame_top_B: type fixed, parent world, child frame_top_B, origin xyz=0.4125 -0.325 0.1375 rpy=0 0 -1.5707963267948966
- added joint world_to_frame_top_F: type fixed, parent world, child frame_top_F, origin xyz=-0.0125 -0.325 0.1375 rpy=0 0 -1.5707963267948966
- added joint world_to_frame_top_L: type fixed, parent world, child frame_top_L, origin xyz=0.20 0.0125 0.1375 rpy=0 0 0
- added joint world_to_frame_top_R: type fixed, parent world, child frame_top_R, origin xyz=0.20 -0.6625 0.1375 rpy=0 0 0
- added joint world_to_frame_vertical_LB: type fixed, parent world, child frame_vertical_LB, origin xyz=0.4125 0.0125 0.075 rpy=0 -1.5707963267948966 0
- added joint world_to_frame_vertical_LF: type fixed, parent world, child frame_vertical_LF, origin xyz=-0.0125 0.0125 0.075 rpy=0 -1.5707963267948966 0
- added joint world_to_frame_vertical_RB: type fixed, parent world, child frame_vertical_RB, origin xyz=0.4125 -0.6625 0.075 rpy=0 -1.5707963267948966 0
- added joint world_to_frame_vertical_RF: type fixed, parent world, child frame_vertical_RF, origin xyz=-0.0125 -0.6625 0.075 rpy=0 -1.5707963267948966 0
- joint base_mount_R: origin xyz=-.2 0 0 rpy=0 0 1.5707963267948966 -> xyz=-0.14858 0.002 0 rpy=0 0 1.5707963267948966
