Commit message: lots of updates

File: raven_2_params/data/ravenII_2arm.original.urdf (robot description, URDF)
Before this commit: robot raven_2, 17 links, 16 joints
Links:
- link base_link_L: geometry visual mesh filename=package://raven_2_params/data/left_arm/base_w_motors.dae
- link base_link_R: geometry visual mesh filename=package://raven_2_params/data/right_arm/base_w_motors.dae
- link grasper1_L: geometry visual mesh filename=package://raven_2_params/data/left_arm/grasper_1.dae
- link grasper1_R: geometry visual mesh filename=package://raven_2_params/data/right_arm/grasper_1.dae
- link grasper2_L: geometry visual mesh filename=package://raven_2_params/data/left_arm/grasper_2.dae
- link grasper2_R: geometry visual mesh filename=package://raven_2_params/data/right_arm/grasper_2.dae
- link instrument_shaft_L: geometry visual mesh filename=package://raven_2_params/data/left_arm/instrument_shaft.dae
- link instrument_shaft_R: geometry visual mesh filename=package://raven_2_params/data/right_arm/instrument_shaft.dae
- link link1_L: geometry visual mesh filename=package://raven_2_params/data/left_arm/link1_w_cover.dae
- link link1_R: geometry visual mesh filename=package://raven_2_params/data/right_arm/link1_w_cover.dae
- link link2_L: geometry visual mesh filename=package://raven_2_params/data/left_arm/link2.dae
- link link2_R: geometry visual mesh filename=package://raven_2_params/data/right_arm/link2.dae
- link link3_L: geometry visual mesh filename=package://raven_2_params/data/left_arm/link3.dae
- link link3_R: geometry visual mesh filename=package://raven_2_params/data/right_arm/link3.dae
- link wrist_L: geometry visual mesh filename=package://raven_2_params/data/left_arm/wrist.dae
- link wrist_R: geometry visual mesh filename=package://raven_2_params/data/right_arm/wrist.dae

File: raven_2_params/data/ravenII_both_arm.urdf (robot description, URDF)
Before this commit: robot raven_2, 28 links, 27 joints
Links:
- added link frame_base_support_L; visual box size=0.4 0.05 0.025
- added link frame_base_support_R; visual box size=0.4 0.05 0.025
- added link frame_bottom_B; visual box size=0.70 0.025 0.025
- added link frame_bottom_F; visual box size=0.7 0.025 0.025
- added link frame_bottom_L; visual box size=0.40 0.025 0.025
- added link frame_bottom_R; visual box size=0.40 0.025 0.025
- added link frame_top_B; visual box size=0.70 0.025 0.025
- added link frame_top_F; visual box size=0.7 0.025 0.025
- added link frame_top_L; visual box size=0.40 0.025 0.025
- added link frame_top_R; visual box size=0.40 0.025 0.025
- added link frame_vertical_LB; visual box size=0.10 0.025 0.025
- added link frame_vertical_LF; visual box size=0.10 0.025 0.025
- added link frame_vertical_RB; visual box size=0.10 0.025 0.025
- added link frame_vertical_RF; visual box size=0.10 0.025 0.025
- link base_link_R: geometry visual mesh filename=package://raven_2_params/data/right_arm/base_w_motors.dae
Joints:
- removed joint tool_base_to_main_L
- removed joint tool_base_to_main_R
- removed joint tool_base_to_tip_L
- removed joint tool_base_to_tip_R
- added joint frame_pose_base_support_L: type fixed, parent world, child frame_base_support_L, origin xyz=0.1315 0.05 0.2 rpy=0 -1.5707963267948966 0
- added joint frame_pose_base_support_R: type fixed, parent world, child frame_base_support_R, origin xyz=0.1315 -0.7 0.2 rpy=0 -1.5707963267948966 0
- added joint frame_pose_bottom_B: type fixed, parent world, child frame_bottom_B, origin xyz=0.4125 -0.325 0.0125 rpy=0 0 -1.5707963267948966
- added joint frame_pose_bottom_F: type fixed, parent world, child frame_bottom_F, origin xyz=-0.0125 -0.325 0.0125 rpy=0 0 -1.5707963267948966
- added joint frame_pose_bottom_L: type fixed, parent world, child frame_bottom_L, origin xyz=0.20 0.0125 0.0125 rpy=0 0 0
- added joint frame_pose_bottom_R: type fixed, parent world, child frame_bottom_R, origin xyz=0.20 -0.6625 0.0125 rpy=0 0 0
- added joint frame_pose_top_B: type fixed, parent world, child frame_top_B, origin xyz=0.4125 -0.325 0.1375 rpy=0 0 -1.5707963267948966
- added joint frame_pose_top_F: type fixed, parent world, child frame_top_F, origin xyz=-0.0125 -0.325 0.1375 rpy=0 0 -1.5707963267948966
- added joint frame_pose_top_L: type fixed, parent world, child frame_top_L, origin xyz=0.20 0.0125 0.1375 rpy=0 0 0
- added joint frame_pose_top_R: type fixed, parent world, child frame_top_R, origin xyz=0.20 -0.6625 0.1375 rpy=0 0 0
- added joint frame_pose_vertical_LB: type fixed, parent world, child frame_vertical_LB, origin xyz=0.4125 0.0125 0.075 rpy=0 -1.5707963267948966 0
- added joint frame_pose_vertical_LF: type fixed, parent world, child frame_vertical_LF, origin xyz=-0.0125 0.0125 0.075 rpy=0 -1.5707963267948966 0
- added joint frame_pose_vertical_RB: type fixed, parent world, child frame_vertical_RB, origin xyz=0.4125 -0.6625 0.075 rpy=0 -1.5707963267948966 0
- added joint frame_pose_vertical_RF: type fixed, parent world, child frame_vertical_RF, origin xyz=-0.0125 -0.6625 0.075 rpy=0 -1.5707963267948966 0
- added joint tool_base_to_tool_L: type fixed, parent tool_base_L, child tool_L, origin xyz=0.01 0 0 rpy=0 0 0, limit lower=0.0 upper=3.1415 effort=1000.0 velocity=0.5
- added joint tool_base_to_tool_R: type fixed, parent tool_base_R, child tool_R, origin xyz=0.01 0 0 rpy=0 0 0, limit lower=0.0 upper=3.1415 effort=1000.0 velocity=0.5
- added joint tool_base_to_tool_tip_L: type fixed, parent tool_base_L, child tool_tip_L, origin xyz=0.02 0 0 rpy=0 0 0, limit lower=0.0 upper=3.1415 effort=1000.0 velocity=0.5
- added joint tool_base_to_tool_tip_R: type fixed, parent tool_base_R, child tool_tip_R, origin xyz=0.02 0 0 rpy=0 0 0, limit lower=0.0 upper=3.1415 effort=1000.0 velocity=0.5
- joint base_mount_R: origin xyz=-.2 0 0 rpy=0 0 1.5707963267948966 -> xyz=-0.14858 0.002 0 rpy=0 0 1.5707963267948966
- joint grasper_joint_1_L: origin xyz=0.012 0 0 rpy=1.5707963267948966 0 0 -> xyz=0.012 0 0 rpy=-1.5707963267948966 0 0
- joint grasper_joint_2_L: origin xyz=0.012 0 0 rpy=1.5707963267948966 0 0 -> xyz=0.012 0 0 rpy=-1.5707963267948966 0 0
- joint tool_roll_L: origin xyz=0 0 0 rpy=0 0 0 -> xyz=0 0 0 rpy=0 0 -3.141592653589793
- joint tool_roll_R: origin xyz=0 0 0 rpy=0 0 -0.37732519171346124 -> xyz=0 0 0 rpy=0 0 -1.5707963267948966
- joint wrist_joint_L: axis 0 0 1 -> 0 0 -1; origin xyz=0 0 0 rpy=-1.5707963267948966 -1.0471975511965979 1.5707963267948966 -> xyz=0 0 0 rpy=1.5707963267948966 -1.5707963267948966 1.5707963267948966

File: raven_2_params/data/ravenII_gold_arm.urdf (robot description, URDF)
Before this commit: robot raven_2, 15 links, 14 joints
Links:
- added link frame_base_support_L; visual box size=0.4 0.05 0.025
- added link frame_base_support_R; visual box size=0.4 0.05 0.025
- added link frame_bottom_B; visual box size=0.70 0.025 0.025
- added link frame_bottom_F; visual box size=0.7 0.025 0.025
- added link frame_bottom_L; visual box size=0.40 0.025 0.025
- added link frame_bottom_R; visual box size=0.40 0.025 0.025
- added link frame_top_B; visual box size=0.70 0.025 0.025
- added link frame_top_F; visual box size=0.7 0.025 0.025
- added link frame_top_L; visual box size=0.40 0.025 0.025
- added link frame_top_R; visual box size=0.40 0.025 0.025
- added link frame_vertical_LB; visual box size=0.10 0.025 0.025
- added link frame_vertical_LF; visual box size=0.10 0.025 0.025
- added link frame_vertical_RB; visual box size=0.10 0.025 0.025
- added link frame_vertical_RF; visual box size=0.10 0.025 0.025
- link base_link_L: geometry visual mesh filename=package://raven_2_params/data/left_arm/base_w_motors.dae
Joints:
- removed joint tool_base_to_main_L
- removed joint tool_base_to_tip_L
- added joint frame_pose_base_support_L: type fixed, parent world, child frame_base_support_L, origin xyz=0.1315 0.05 0.2 rpy=0 -1.5707963267948966 0
- added joint frame_pose_base_support_R: type fixed, parent world, child frame_base_support_R, origin xyz=0.1315 -0.7 0.2 rpy=0 -1.5707963267948966 0
- added joint frame_pose_bottom_B: type fixed, parent world, child frame_bottom_B, origin xyz=0.4125 -0.325 0.0125 rpy=0 0 -1.5707963267948966
- added joint frame_pose_bottom_F: type fixed, parent world, child frame_bottom_F, origin xyz=-0.0125 -0.325 0.0125 rpy=0 0 -1.5707963267948966
- added joint frame_pose_bottom_L: type fixed, parent world, child frame_bottom_L, origin xyz=0.20 0.0125 0.0125 rpy=0 0 0
- added joint frame_pose_bottom_R: type fixed, parent world, child frame_bottom_R, origin xyz=0.20 -0.6625 0.0125 rpy=0 0 0
- added joint frame_pose_top_B: type fixed, parent world, child frame_top_B, origin xyz=0.4125 -0.325 0.1375 rpy=0 0 -1.5707963267948966
- added joint frame_pose_top_F: type fixed, parent world, child frame_top_F, origin xyz=-0.0125 -0.325 0.1375 rpy=0 0 -1.5707963267948966
- added joint frame_pose_top_L: type fixed, parent world, child frame_top_L, origin xyz=0.20 0.0125 0.1375 rpy=0 0 0
- added joint frame_pose_top_R: type fixed, parent world, child frame_top_R, origin xyz=0.20 -0.6625 0.1375 rpy=0 0 0
- added joint frame_pose_vertical_LB: type fixed, parent world, child frame_vertical_LB, origin xyz=0.4125 0.0125 0.075 rpy=0 -1.5707963267948966 0
- added joint frame_pose_vertical_LF: type fixed, parent world, child frame_vertical_LF, origin xyz=-0.0125 0.0125 0.075 rpy=0 -1.5707963267948966 0
- added joint frame_pose_vertical_RB: type fixed, parent world, child frame_vertical_RB, origin xyz=0.4125 -0.6625 0.075 rpy=0 -1.5707963267948966 0
- added joint frame_pose_vertical_RF: type fixed, parent world, child frame_vertical_RF, origin xyz=-0.0125 -0.6625 0.075 rpy=0 -1.5707963267948966 0
- added joint tool_base_to_tool_L: type fixed, parent tool_base_L, child tool_L, origin xyz=0.01 0 0 rpy=0 0 0, limit lower=0.0 upper=3.1415 effort=1000.0 velocity=0.5
- added joint tool_base_to_tool_tip_L: type fixed, parent tool_base_L, child tool_tip_L, origin xyz=0.02 0 0 rpy=0 0 0, limit lower=0.0 upper=3.1415 effort=1000.0 velocity=0.5
- joint grasper_joint_1_L: origin xyz=0.012 0 0 rpy=1.5707963267948966 0 0 -> xyz=0.012 0 0 rpy=-1.5707963267948966 0 0
- joint grasper_joint_2_L: origin xyz=0.012 0 0 rpy=1.5707963267948966 0 0 -> xyz=0.012 0 0 rpy=-1.5707963267948966 0 0
- joint tool_roll_L: origin xyz=0 0 0 rpy=0 0 0 -> xyz=0 0 0 rpy=0 0 -3.141592653589793
- joint wrist_joint_L: axis 0 0 1 -> 0 0 -1; origin xyz=0 0 0 rpy=-1.5707963267948966 -1.0471975511965979 1.5707963267948966 -> xyz=0 0 0 rpy=1.5707963267948966 -1.5707963267948966 1.5707963267948966

File: raven_2_params/data/ravenII_green_arm.urdf (robot description, URDF)
Before this commit: robot raven_2, 30 links, 29 joints
Links:
- removed link base_link_L
Joints:
- removed joint base_mount_L
- removed joint tool_base_to_main_R
- removed joint tool_base_to_tip_R
- removed joint world_to_frame_base_support_L
- removed joint world_to_frame_base_support_R
- removed joint world_to_frame_bottom_B
- removed joint world_to_frame_bottom_F
- removed joint world_to_frame_bottom_L
- removed joint world_to_frame_bottom_R
- removed joint world_to_frame_top_B
- removed joint world_to_frame_top_F
- removed joint world_to_frame_top_L
- removed joint world_to_frame_top_R
- removed joint world_to_frame_vertical_LB
- removed joint world_to_frame_vertical_LF
- removed joint world_to_frame_vertical_RB
- removed joint world_to_frame_vertical_RF
- added joint frame_pose_base_support_L: type fixed, parent world, child frame_base_support_L, origin xyz=0.1315 0.05 0.2 rpy=0 -1.5707963267948966 0
- added joint frame_pose_base_support_R: type fixed, parent world, child frame_base_support_R, origin xyz=0.1315 -0.7 0.2 rpy=0 -1.5707963267948966 0
- added joint frame_pose_bottom_B: type fixed, parent world, child frame_bottom_B, origin xyz=0.4125 -0.325 0.0125 rpy=0 0 -1.5707963267948966
- added joint frame_pose_bottom_F: type fixed, parent world, child frame_bottom_F, origin xyz=-0.0125 -0.325 0.0125 rpy=0 0 -1.5707963267948966
- added joint frame_pose_bottom_L: type fixed, parent world, child frame_bottom_L, origin xyz=0.20 0.0125 0.0125 rpy=0 0 0
- added joint frame_pose_bottom_R: type fixed, parent world, child frame_bottom_R, origin xyz=0.20 -0.6625 0.0125 rpy=0 0 0
- added joint frame_pose_top_B: type fixed, parent world, child frame_top_B, origin xyz=0.4125 -0.325 0.1375 rpy=0 0 -1.5707963267948966
- added joint frame_pose_top_F: type fixed, parent world, child frame_top_F, origin xyz=-0.0125 -0.325 0.1375 rpy=0 0 -1.5707963267948966
- added joint frame_pose_top_L: type fixed, parent world, child frame_top_L, origin xyz=0.20 0.0125 0.1375 rpy=0 0 0
- added joint frame_pose_top_R: type fixed, parent world, child frame_top_R, origin xyz=0.20 -0.6625 0.1375 rpy=0 0 0
- added joint frame_pose_vertical_LB: type fixed, parent world, child frame_vertical_LB, origin xyz=0.4125 0.0125 0.075 rpy=0 -1.5707963267948966 0
- added joint frame_pose_vertical_LF: type fixed, parent world, child frame_vertical_LF, origin xyz=-0.0125 0.0125 0.075 rpy=0 -1.5707963267948966 0
- added joint frame_pose_vertical_RB: type fixed, parent world, child frame_vertical_RB, origin xyz=0.4125 -0.6625 0.075 rpy=0 -1.5707963267948966 0
- added joint frame_pose_vertical_RF: type fixed, parent world, child frame_vertical_RF, origin xyz=-0.0125 -0.6625 0.075 rpy=0 -1.5707963267948966 0
- added joint tool_base_to_tool_R: type fixed, parent tool_base_R, child tool_R, origin xyz=0.01 0 0 rpy=0 0 0, limit lower=0.0 upper=3.1415 effort=1000.0 velocity=0.5
- added joint tool_base_to_tool_tip_R: type fixed, parent tool_base_R, child tool_tip_R, origin xyz=0.02 0 0 rpy=0 0 0, limit lower=0.0 upper=3.1415 effort=1000.0 velocity=0.5
- joint tool_roll_R: origin xyz=0 0 0 rpy=0 0 -0.37732519171346124 -> xyz=0 0 0 rpy=0 0 -1.5707963267948966
